File: electronics/cnc-controller/cnc-controller.sch (EAGLE design)
At the start: 116 parts, among them Q1 MOSFET-NCHANNELSMD, Q10 BSS84, Q11 BSS84, Q12 BSS84, Q13 BSS84, Q14 BSS84, Q15 BSS84, Q16 BSS84, Q17 BSS84, Q18 BSS84, Q19 BSS84, Q2 MOSFET-NCHANNELSMD, Q20 BSS84, Q21 BSS84, Q3 MOSFET-NCHANNELSMD, Q7 BSS84, Q8 BSS84, Q9 BSS84, U1 MCP41XXX, U16 USD-SOCKETNEW, X1 MSTBA2

Commit message: updated cnc driver shield and various tweaks to milling config.
Parts:
- removed DPOT, RELAY: CONN-3XH-3, Hoektronics:CONN-3XH-3
- removed INTERFACE: CONN-12, Hoektronics:CONN-12
- removed Q2: MOSFET-NCHANNELSMD, SparkFun:MOSFET-NCHANNELSMD
- removed R2, R9: 100k, Hoektronics:RESISTOR0603
- removed R62, R63: 330, Hoektronics:RESISTOR0603
- removed U1: MCP41XXX, Hoektronics:MCP41XXX
- added C11, C12, C13: (no value), Hoektronics:CAPACITOR0805
- added ENCODER: CONN-5, Hoektronics:CONN-5
- added LCD: CONN-16, Hoektronics:CONN-16
- added Q4: BSS84, SparkFun:MOSFET-NCHANNELSMD
- added R15, R7, R8: 1k, Hoektronics:RESISTOR0805
- added R19, R23: 100k, Hoektronics:RESISTOR0603
- added R21, R26: 330, Hoektronics:RESISTOR0603
- added R6: (no value), pot:TRIM_US-B25P
- added SPINDLE: CONN-3XH-3, Hoektronics:CONN-3XH-3
- Q3: value MOSFET-NCHANNELSMD -> BSS84
- VACUUM: value CONN-2 -> CONN-3XH-3; device Hoektronics:CONN-2 -> Hoektronics:CONN-3XH-3
Connections:
- removed net CANCEL_PIN: INTERFACE.10, U$1.D14
- removed net MENU_PIN: INTERFACE.11, U$1.D15
- removed net N$34: DPOT.1, U1.PB0
- removed net N$36: DPOT.3, U1.PA0
- removed net N$6: DPOT.2, U1.PW0
- removed net N$60: Q2.G, R62.1, R9.2
- removed net N$61: Q3.G, R2.2, R63.1
- removed net N$62: Q3.D, RELAY.2
- removed net N$63: Q2.D, VACUUM.2
- new net ENC_A_PIN: C12.1, ENCODER.2, R8.1, U$1.D14
- new net ENC_B_PIN: C13.1, ENCODER.3, R15.1, U$1.D15
- new net N$1: LCD.3, R6.S
- new net N$10: Q3.G, R19.2, R21.1
- new net N$11: Q4.G, R23.2, R26.1
- new net N$12: Q3.D, VACUUM.3
- new net N$13: Q4.D, SPINDLE.3
- net 5V: no longer RELAY.1, VACUUM.1
- net DEBUG_LED: no longer INTERFACE.12
- net DIGIPOT_SELECT: no longer U1.CS
- net GND: now also C11.2, C12.2, C13.2, ENCODER.4, ENCODER.5, LCD.1, LCD.16, LCD.5, Q4.S, R19.1, R23.1, R6.A, SPINDLE.2, VACUUM.2; no longer INTERFACE.1, Q2.S, R2.1, R9.1, RELAY.3, U1.VSS
- net LCD_D4: now also LCD.11; no longer INTERFACE.8
- net LCD_D5: now also LCD.12; no longer INTERFACE.7
- net LCD_D6: now also LCD.13; no longer INTERFACE.6
- net LCD_D7: now also LCD.14; no longer INTERFACE.5
- net LCD_EN: now also LCD.6; no longer INTERFACE.4
- net LCD_RS: now also LCD.4; no longer INTERFACE.3
- net MOSI: no longer U1.SI
- net OK_PIN: now also C11.1, ENCODER.1, R7.1; no longer INTERFACE.9
- net SCK: no longer U1.SCK
- net SPINDLE: now also R26.2; no longer R63.2
- net VACUUM: now also R21.2; no longer R62.2
- net VCC: now also LCD.15, LCD.2, R15.2, R6.E, R7.2, R8.2, SPINDLE.1, VACUUM.1; no longer INTERFACE.2, U1.VDD
Other:
- note added: "12V RGB LEDS"
- note added: "20x4 LCD"
- note added: "24V DC OUT"
- note added: "Copyright 2014 Hoektronics.com"
- note added: "Encoder"
- note added: "Revision E"
- note added: "SPINDLE"
- note added: "Spindle Driver"
- note added: "Spindle Tach"
- note added: "VACUUM"
- note removed: "12-40V DC OUT"
- note removed: "12V RGB LED STRIP"
- note removed: "Copyright 2012 Hoektronics.com"
- note removed: "External Relay Circuits"
- note removed: "LCD"
- note removed: "Revision C"
- note removed: "Spindle Relay"
- note removed: "Spindle Speed Output"
- note removed: "Vacuum Relay"

Commit message: a few more cleanups before the Rev E release.
Other:
- note removed: "HOLES"
